Commit message: Edited friction values of wheels

File: volta_description/urdf/components/wheel_volta.urdf.xacro (robot description, xacro)
@@ -30,7 +30,7 @@
         <link name="${wheel_prefix}_wheel">
             <visual>
-                <origin xyz="0 0 0" rpy="0 0 0"/>
+                <origin xyz="0 0 0" rpy="1.57 0 0"/>
                 <geometry>
-                    <mesh filename="package://volta_description/meshes/wheel_volta.STL"/>
+                    <cylinder length="${wheel_width}" radius="${wheel_radius}"/>
                 </geometry>
                 <material name="black"/>
@@ -43,17 +43,9 @@
             </collision>
             <inertial>
-                <mass value="2.637" />
-                <origin xyz="0 0 0" />
+                <mass value="0.050" />
+                <origin xyz="0 0 0" rpy="0 0 0" />
                 <inertia  ixx="${wheel_ixx}" ixy="${wheel_ixy}" ixz="${wheel_ixz}" iyy="${wheel_iyy}" iyz="${wheel_iyz}" izz="${wheel_izz}" />
             </inertial>
         </link>
-        <gazebo reference="${wheel_prefix}_wheel">
-            <material>Gazebo/Black</material>
-            <mu1 value="1.0"/>
-            <mu2 value="1.0"/>
-            <kp value="10000000.0"></kp>
-            <kd value="1.0"></kd>
-            <fdir1 value="1 0 0"/>
-        </gazebo>
         <!-- Wheel Joint -->
         <joint name="${wheel_prefix}_wheel_joint" type="continuous">
@@ -62,4 +54,5 @@
             <xacro:insert_block name="joint_origin" />
             <axis xyz="0 1 0" />
+	    <anchor xyz="0 0 0"/>
         </joint>
         <!-- Wheel Transmission -->

File: volta_description/urdf/volta.urdf.xacro (robot description, xacro)
@@ -61,4 +61,5 @@
             </collision>
             <inertial>
+		<origin xyz ="-0.0223 0.0000 0.1018"/>
                 <mass value="${base_mass}"/>
                 <inertia ixx="${base_ixx}" ixy="${base_ixy}" ixz="${base_ixz}" iyy="${base_iyy}" iyz="${base_iyz}" izz="${base_izz}"/>

File: volta_description/urdf/volta_properties.xacro (robot description, xacro)
@@ -35,25 +35,33 @@
     </material>
     <xacro:property name="base_underside_h" value="0.03275"/>
-    <xacro:property name="base_mass" value="200.0000"/>
+    <xacro:property name="base_mass" value="15.0000"/>
     <xacro:property name="base_l" value="0.4000"/>
     <xacro:property name="base_w" value="0.3200"/>
     <xacro:property name="base_h" value="0.2295"/>
-    <xacro:property name="base_ixx" value="3.0"/>
-    <xacro:property name="base_ixy" value="0.0040"/>
-    <xacro:property name="base_ixz" value="0.0043"/>
-    <xacro:property name="base_iyy" value="3.0"/>
-    <xacro:property name="base_iyz" value="0.0001"/>
-    <xacro:property name="base_izz" value="0.1945"/>
-    <xacro:property name="wheel_mass" value="0.100"/>
+    <!--
+    <xacro:property name="base_ixx" value="0.3426"/>
+    <xacro:property name="base_ixy" value="0.0000"/>
+    <xacro:property name="base_ixz" value="-0.0503"/>
+    <xacro:property name="base_iyy" value="0.3917"/>
+    <xacro:property name="base_iyz" value="0.0000"/>
+    <xacro:property name="base_izz" value="0.3001"/>
+    -->
+    <xacro:property name="base_ixx" value="0.1815"/>
+    <xacro:property name="base_ixy" value="0.0000"/>
+    <xacro:property name="base_ixz" value="-0.0158"/>
+    <xacro:property name="base_iyy" value="0.2238"/>
+    <xacro:property name="base_iyz" value="0.0000"/>
+    <xacro:property name="base_izz" value="0.2856"/>
+    <xacro:property name="wheel_mass" value="0.0563"/>
     <xacro:property name="wheel_width" value="0.020" />
     <xacro:property name="wheel_radius" value="0.034" />
     <xacro:property name="wheel_joint_y_abs" value="0.1425" />
     <xacro:property name="wheel_joint_z_abs" value="0.0215" />
-    <xacro:property name="wheel_ixx" value="0.739"/>
-    <xacro:property name="wheel_ixy" value="0.170"/>
-    <xacro:property name="wheel_ixz" value="0.236"/>
-    <xacro:property name="wheel_iyy" value="0.741"/>
-    <xacro:property name="wheel_iyz" value="0.299"/>
-    <xacro:property name="wheel_izz" value="0.460"/>
+    <xacro:property name="wheel_ixx" value="0.001"/>
+    <xacro:property name="wheel_ixy" value="0.000"/>
+    <xacro:property name="wheel_ixz" value="0.000"/>
+    <xacro:property name="wheel_iyy" value="0.001"/>
+    <xacro:property name="wheel_iyz" value="0.000"/>
+    <xacro:property name="wheel_izz" value="0.001"/>
     <xacro:property name="caster_radius" value="0.016"/>
     <xacro:property name="caster_joint_x" value="0.1200"/>

Commit message: Updated Friction Values in URDF

File: volta_description/urdf/components/wheel_volta.urdf.xacro (robot description, xacro)
@@ -30,5 +30,5 @@
         <link name="${wheel_prefix}_wheel">
             <visual>
-                <origin xyz="0 0 0" rpy="1.57 0 0"/>
+                <origin xyz="0 0 0" rpy="1.57159 0 0"/>
                 <geometry>
                     <cylinder length="${wheel_width}" radius="${wheel_radius}"/>
@@ -37,5 +37,5 @@
             </visual>
             <collision>
-                <origin xyz="0 0 0" rpy="1.57 0 0"/>
+                <origin xyz="0 0 0" rpy="1.57159 0 0"/>
                 <geometry>
                     <cylinder length="${wheel_width}" radius="${wheel_radius}" />
@@ -48,4 +48,12 @@
             </inertial>
         </link>
+        <gazebo reference="${wheel_prefix}_wheel">
+            <material>Gazebo/Black</material>
+            <mu1 value="1"/>
+            <mu2 value="1"/>
+            <kp value="10000000.0"></kp>
+            <kd value="1.0"></kd>
+            <fdir1 value="1 0 0"/>
+        </gazebo>
         <!-- Wheel Joint -->
         <joint name="${wheel_prefix}_wheel_joint" type="continuous">
@@ -54,5 +62,5 @@
             <xacro:insert_block name="joint_origin" />
             <axis xyz="0 1 0" />
-	    <anchor xyz="0 0 0"/>
+            <anchor xyz="0 0 0"/>
         </joint>
         <!-- Wheel Transmission -->

File: volta_description/urdf/volta.urdf.xacro (robot description, xacro)
@@ -34,5 +34,5 @@
     <xacro:arg name="tf_pre" default="" />
     <xacro:arg name="lidar_enabled" default="true"/>
-    <xacro:arg name="imu_enabled" default="false"/>
+    <xacro:arg name="imu_enabled" default="true"/>
     <xacro:arg name="camera_enabled" default="true"/>
     <xacro:macro name="volta_robot">
@@ -61,5 +61,5 @@
             </collision>
             <inertial>
-		<origin xyz ="-0.0223 0.0000 0.1018"/>
+                <origin xyz ="-0.0223 0.0000 0.1018"/>
                 <mass value="${base_mass}"/>
                 <inertia ixx="${base_ixx}" ixy="${base_ixy}" ixz="${base_ixz}" iyy="${base_iyy}" iyz="${base_iyz}" izz="${base_izz}"/>
@@ -100,4 +100,6 @@
         <gazebo reference="caster_front_left_link">
             <turnGravityOff>false</turnGravityOff>
+            <mu1 value="0.0"/>
+            <mu2 value="0.0"/>
         </gazebo>
         <link name="caster_front_right_link">
@@ -128,4 +130,6 @@
         <gazebo reference="caster_front_right_link">
             <turnGravityOff>false</turnGravityOff>
+            <mu1 value="0.0"/>
+            <mu2 value="0.0"/>
         </gazebo>
         <link name="caster_rear_right_link">
@@ -156,4 +160,6 @@
         <gazebo reference="caster_rear_right_link">
             <turnGravityOff>false</turnGravityOff>
+            <mu1 value="0.0"/>
+            <mu2 value="0.0"/>
         </gazebo>
         <link name="caster_rear_left_link">
@@ -184,4 +190,6 @@
         <gazebo reference="caster_rear_left_link">
             <turnGravityOff>false</turnGravityOff>
+            <mu1 value="0.0"/>
+            <mu2 value="0.0"/>
         </gazebo>
         <gazebo>

File: volta_description/urdf/volta_properties.xacro (robot description, xacro)
@@ -39,12 +39,4 @@
     <xacro:property name="base_w" value="0.3200"/>
     <xacro:property name="base_h" value="0.2295"/>
-    <!--
-    <xacro:property name="base_ixx" value="0.3426"/>
-    <xacro:property name="base_ixy" value="0.0000"/>
-    <xacro:property name="base_ixz" value="-0.0503"/>
-    <xacro:property name="base_iyy" value="0.3917"/>
-    <xacro:property name="base_iyz" value="0.0000"/>
-    <xacro:property name="base_izz" value="0.3001"/>
-    -->
     <xacro:property name="base_ixx" value="0.1815"/>
     <xacro:property name="base_ixy" value="0.0000"/>
