Commit message: inclusion of sensors on demo unit

File: volta_description/urdf/accessories/rpi_a3_volta.urdf.xacro (robot description, xacro)
@@ -28,5 +28,5 @@
                  min_angle:=-1.57 max_angle:=1.57 min_range:=0.5 max_range:=10.0 robot_namespace:=/">
       <joint name="lidar_joint" type="fixed">
-          <origin xyz="${lidar_joint_x} ${lidar_joint_y} ${lidar_joint_z}" rpy="0 0 0" />
+          <origin xyz="${lidar_joint_x} ${lidar_joint_y} ${lidar_joint_z}" rpy="0 0 3.14159" />
           <parent link="base_link" />
           <child link="${frame}" />

Commit message: Adding in of URG_node

File: volta_description/urdf/accessories/rpi_a3_volta.urdf.xacro (robot description, xacro)
@@ -28,5 +28,5 @@
                  min_angle:=-1.57 max_angle:=1.57 min_range:=0.5 max_range:=10.0 robot_namespace:=/">
       <joint name="lidar_joint" type="fixed">
-          <origin xyz="${lidar_joint_x} ${lidar_joint_y} ${lidar_joint_z}" rpy="0 0 3.14159" />
+          <origin xyz="${lidar_joint_x} ${lidar_joint_y} ${lidar_joint_z}" rpy="0 0 0" />
           <parent link="base_link" />
           <child link="${frame}" />
