Commit message: inclusion of the URDF file format for the Camera_link

File: volta_description/urdf/accessories/camera_volta.urdf.xacro (robot description, xacro)
@@ -51,4 +51,10 @@
             </inertial>
         </link>
+        <joint name="trans_joint" type="fixed">
+               <origin xyz="0 0 0" rpy="0 0 0 "/>
+               <parent link="${frame}"/>
+               <child link="camera_link"/>
+        </joint>
+        <link name="camera_link"> </link>
         <gazebo reference="${frame}">
             <sensor type="camera" name="camera">
@@ -71,18 +77,29 @@
                     </noise>
                 </camera>
-                <plugin name="camera_controller" filename="libgazebo_ros_camera.so">
+                <plugin name="camera_controller" filename="libgazebo_ros_openni_kinetic.so">
                     <!-- <robotNamespace>${robot_namespace}</robotNamespace> -->
+                    <baseline>0.2</baseline>
                     <alwaysOn>true</alwaysOn>
-                    <updateRate>${update_rate}</updateRate>
-                    <cameraName>${frame}</cameraName>
-                    <imageTopicName>${topic}</imageTopicName>
-                    <cameraInfoTopicName>${info_topic}</cameraInfoTopicName>
-                    <frameName>${frame}</frameName>
-                    <hackBaseline>0.07</hackBaseline>
-                    <distortionK1>0.0</distortionK1>
-                    <distortionK2>0.0</distortionK2>
-                    <distortionK3>0.0</distortionK3>
-                    <distortionT1>0.0</distortionT1>
-                    <distortionT2>0.0</distortionT2>
+                        <updateRate>${update_rate}</updateRate>
+                        <cameraName>${frame}</cameraName>
+                        <frameName>camera_link</frameName>
+                    <imageTopicName>${topic}/color/image_raw</imageTopicName>
+                    <cameraInfoTopicName>${topic}/color/camera_info</cameraInfoTopicName>
+                    <depthImageTopicName>/${topic}/depth/image_raw</depthImageTopicName>
+                    <depthImageInfoTopicName>/${topic}/depth/camera_info</depthImageInfoTopicName>
+                    <pointCloudTopicName>/${topic}/depth/points</pointCloudTopicName>
+                    <pointCloudCutoff>0.5</pointCloudCutoff>
+                    <pointCloudCutoffMax>3.0</pointCloudCutoffMax>
+                        <hackBaseline>0.07</hackBaseline>
+                        <distortionK1>0.0</distortionK1>
+                        <distortionK2>0.0</distortionK2>
+                        <distortionK3>0.0</distortionK3>
+                        <distortionT1>0.0</distortionT1>
+                        <distortionT2>0.0</distortionT2>
+                    <CxPrime>0</CxPrime>
+                    <Cx>0</Cx>
+                    <Cy>0</Cy>
+                    <focalLength>0</focalLength>
+                    <hackBaseline>0</hackBaseline>
                 </plugin>
             </sensor>

Commit message: Update camera_volta.urdf.xacro

File: volta_description/urdf/accessories/camera_volta.urdf.xacro (robot description, xacro)
@@ -51,5 +51,5 @@
             </inertial>
         </link>
-        <joint name="trans_joint" type="fixed">
+        <joint name="camera_transformation_joint" type="fixed">
                <origin xyz="0 0 0" rpy="0 0 0 "/>
                <parent link="${frame}"/>

Commit message: Updated Wheel Radius, Camera Plugin Frame

File: volta_description/urdf/accessories/camera_volta.urdf.xacro (robot description, xacro)
@@ -51,10 +51,4 @@
             </inertial>
         </link>
-        <joint name="camera_transformation_joint" type="fixed">
-               <origin xyz="0 0 0" rpy="0 0 0 "/>
-               <parent link="${frame}"/>
-               <child link="camera_link"/>
-        </joint>
-        <link name="camera_link"> </link>
         <gazebo reference="${frame}">
             <sensor type="camera" name="camera">
@@ -83,5 +77,5 @@
                         <updateRate>${update_rate}</updateRate>
                         <cameraName>${frame}</cameraName>
-                        <frameName>camera_link</frameName>
+                        <frameName>${frame}</frameName>
                     <imageTopicName>${topic}/color/image_raw</imageTopicName>
                     <cameraInfoTopicName>${topic}/color/camera_info</cameraInfoTopicName>

File: volta_description/urdf/volta_properties.xacro (robot description, xacro)
@@ -47,5 +47,5 @@
     <xacro:property name="wheel_mass" value="0.0563"/>
     <xacro:property name="wheel_width" value="0.020" />
-    <xacro:property name="wheel_radius" value="0.034" />
+    <xacro:property name="wheel_radius" value="0.035" />
     <xacro:property name="wheel_joint_y_abs" value="0.1425" />
     <xacro:property name="wheel_joint_z_abs" value="0.0215" />
