Commit message: Merged volta_development.

File: volta_description/urdf/accessories/camera_volta.urdf.xacro (robot description, xacro)
@@ -24,31 +24,62 @@
 SOFTWARE, EVEN IF ADVISED OF THE POSSIBILITY OF SUCH DAMAGE.
 -->
-<!-- TODO: Camera Mesh, Mount and Origin -->
 <robot name="volta" xmlns:xacro="https://ros.org/wiki/xacro">
-    <xacro:macro name="camera_" params="frame:=camera topic:=camera info_topic:=camera_info update_rate:=50 robot_namespace:=/">
-        <joint name="base_to_camera" type="fixed">
-            <parent link="base_link"/>
-            <child link="${frame}"/>
-            <origin xyz="${camera_joint_x} ${camera_joint_y} ${camera_joint_z}"/>
-        </joint>
-        <link name="${frame}">
-            <visual>
-                <origin xyz="0 0 0" rpy="0 0 0"/>
-                <geometry>
-                    <mesh filename="package://volta_description/meshes/d435i.STL"/>
-                </geometry>
-            </visual>
-            <collision>
-                <origin xyz="0 0 0" rpy="0 0 0"/>
-                <geometry>
-                    <mesh filename="package://volta_description/meshes/d435i.STL"/>
-                </geometry>
-            </collision>
-            <inertial>
-                <mass value="0.162"/>
-                <origin xyz="0 0 0" rpy="0 0 0"/>
-                <inertia ixx="1.0" ixy="0.0" ixz="0.0" iyy="1.0" iyz="0.0" izz="1.0"/>
-            </inertial>
-        </link>
+    <xacro:macro name="camera_" params="frame:=camera topic:=camera info_topic:=camera_info update_rate:=50 intel_d435i_enabled:=true orbbec_astra_pro_enabled:=false robot_namespace:=/">
+        <xacro:if value="${intel_d435i_enabled}">
+          <!-- Camera link -->
+          <link name="${frame}">
+              <visual>
+                  <origin xyz="0 0 -0.0125" rpy="0 0 0"/>
+                  <geometry>
+                      <mesh filename="package://volta_description/meshes/d435i.dae"/>
+                  </geometry>
+              </visual>
+              <collision>
+                  <origin xyz="0 0 -0.0125" rpy="0 0 0"/>
+                  <geometry>
+                      <mesh filename="package://volta_description/meshes/d435i.dae"/>
+                  </geometry>
+              </collision>
+              <inertial>
+                  <mass value="0.162"/>
+                  <origin xyz="-0.003 0 ${0.0125-0.0125}" rpy="0 0 0"/>
+                  <inertia ixx="0.00011" ixy="0.0" ixz="0.0" iyy="0.00005" iyz="0.0" izz="0.00011"/>
+              </inertial>
+          </link>
+          <!-- Camera joint -->
+          <joint name="base_to_camera" type="fixed">
+              <parent link="base_link"/>
+              <child link="${frame}"/>
+              <origin xyz="${camera_joint_x} ${camera_joint_y} ${camera_joint_z + 0.0125}"/>
+          </joint>
+        </xacro:if>
+        <xacro:if value="${orbbec_astra_pro_enabled}">
+          <!-- Camera link -->
+          <link name="${frame}">
+              <visual>
+                  <origin xyz="0 0 -0.0337" rpy="0 0 0"/>
+                  <geometry>
+                      <mesh filename="package://volta_description/meshes/astra.dae"/>
+                  </geometry>
+              </visual>
+              <collision>
+                  <origin xyz="0 0 -0.0337" rpy="0 0 0"/>
+                  <geometry>
+                      <mesh filename="package://volta_description/meshes/astra.dae"/>
+                  </geometry>
+              </collision>
+              <inertial>
+                  <mass value="0.3"/>
+                  <origin xyz="-0.004 0 ${0.028 - 0.0337}" rpy="0 0 0"/>
+                  <inertia ixx="0.0002" ixy="0.0" ixz="0.0" iyy="0.0003" iyz="0.0" izz="0.0003"/>
+              </inertial>
+          </link>
+          <!-- Camera joint -->
+          <joint name="base_to_camera" type="fixed">
+              <parent link="base_link"/>
+              <child link="${frame}"/>
+              <origin xyz="${camera_joint_x} ${camera_joint_y} ${camera_joint_z + 0.0337}"/>
+          </joint>
+        </xacro:if>
         <gazebo reference="${frame}">
             <sensor type="camera" name="camera">
@@ -71,29 +102,18 @@
                     </noise>
                 </camera>
-                <plugin name="camera_controller" filename="libgazebo_ros_openni_kinetic.so">
+                <plugin name="camera_controller" filename="libgazebo_ros_camera.so">
                     <!-- <robotNamespace>${robot_namespace}</robotNamespace> -->
-                    <baseline>0.2</baseline>
                     <alwaysOn>true</alwaysOn>
-                        <updateRate>${update_rate}</updateRate>
-                        <cameraName>${frame}</cameraName>
-                        <frameName>${frame}</frameName>
-                    <imageTopicName>${topic}/color/image_raw</imageTopicName>
-                    <cameraInfoTopicName>${topic}/color/camera_info</cameraInfoTopicName>
-                    <depthImageTopicName>/${topic}/depth/image_raw</depthImageTopicName>
-                    <depthImageInfoTopicName>/${topic}/depth/camera_info</depthImageInfoTopicName>
-                    <pointCloudTopicName>/${topic}/depth/points</pointCloudTopicName>
-                    <pointCloudCutoff>0.5</pointCloudCutoff>
-                    <pointCloudCutoffMax>3.0</pointCloudCutoffMax>
-                        <hackBaseline>0.07</hackBaseline>
-                        <distortionK1>0.0</distortionK1>
-                        <distortionK2>0.0</distortionK2>
-                        <distortionK3>0.0</distortionK3>
-                        <distortionT1>0.0</distortionT1>
-                        <distortionT2>0.0</distortionT2>
-                    <CxPrime>0</CxPrime>
-                    <Cx>0</Cx>
-                    <Cy>0</Cy>
-                    <focalLength>0</focalLength>
-                    <hackBaseline>0</hackBaseline>
+                    <updateRate>${update_rate}</updateRate>
+                    <cameraName>${frame}</cameraName>
+                    <imageTopicName>${topic}</imageTopicName>
+                    <cameraInfoTopicName>${info_topic}</cameraInfoTopicName>
+                    <frameName>${frame}</frameName>
+                    <hackBaseline>0.07</hackBaseline>
+                    <distortionK1>0.0</distortionK1>
+                    <distortionK2>0.0</distortionK2>
+                    <distortionK3>0.0</distortionK3>
+                    <distortionT1>0.0</distortionT1>
+                    <distortionT2>0.0</distortionT2>
                 </plugin>
             </sensor>

File: volta_description/urdf/components/wheel_volta.urdf.xacro (robot description, xacro)
@@ -30,12 +30,12 @@
         <link name="${wheel_prefix}_wheel">
             <visual>
-                <origin xyz="0 0 0" rpy="1.57159 0 0"/>
+                <origin xyz="0 0 0" rpy="1.570796327 0 0"/>
                 <geometry>
                     <cylinder length="${wheel_width}" radius="${wheel_radius}"/>
                 </geometry>
-                <material name="black"/>
+                <material name="red"/>
             </visual>
             <collision>
-                <origin xyz="0 0 0" rpy="1.57159 0 0"/>
+                <origin xyz="0 0 0" rpy="1.570796327 0 0"/>
                 <geometry>
                     <cylinder length="${wheel_width}" radius="${wheel_radius}" />
@@ -43,5 +43,5 @@
             </collision>
             <inertial>
-                <mass value="0.050" />
+                <mass value="${wheel_mass}" />
                 <origin xyz="0 0 0" rpy="0 0 0" />
                 <inertia  ixx="${wheel_ixx}" ixy="${wheel_ixy}" ixz="${wheel_ixz}" iyy="${wheel_iyy}" iyz="${wheel_iyz}" izz="${wheel_izz}" />
@@ -49,8 +49,8 @@
         </link>
         <gazebo reference="${wheel_prefix}_wheel">
-            <material>Gazebo/Black</material>
-            <mu1 value="1"/>
-            <mu2 value="1"/>
-            <kp value="10000000.0"></kp>
+            <material>Gazebo/Red</material>
+            <mu1 value="1400"/>
+            <mu2 value="600"/>
+            <kp value="3100000.0"></kp>
             <kd value="1.0"></kd>
             <fdir1 value="1 0 0"/>
@@ -62,5 +62,4 @@
             <xacro:insert_block name="joint_origin" />
             <axis xyz="0 1 0" />
-            <anchor xyz="0 0 0"/>
         </joint>
         <!-- Wheel Transmission -->

File: volta_description/urdf/volta.urdf.xacro (robot description, xacro)
@@ -28,12 +28,17 @@
     <xacro:include filename="$(find volta_description)/urdf/volta_properties.xacro"/>
     <xacro:include filename="$(find volta_description)/urdf/components/wheel_volta.urdf.xacro"/>
+    <xacro:include filename="$(find volta_description)/urdf/components/caster_volta.urdf.xacro"/>
     <!-- xacro properties -->
     <xacro:property name="PI" value="3.14159"/>
     <!-- xacro args -->
     <xacro:arg name="robot_namespace" default="/" />
-    <xacro:arg name="tf_pre" default="" />
+    <xacro:arg name="tf_pre" default=""/>
     <xacro:arg name="lidar_enabled" default="true"/>
+    <xacro:arg name="rplidar_a3_enabled" default="true"/>
+    <xacro:arg name="hokuyo_ust_10lx_enabled" default="false"/>
     <xacro:arg name="imu_enabled" default="true"/>
     <xacro:arg name="camera_enabled" default="true"/>
+    <xacro:arg name="intel_d435i_enabled" default="true"/>
+    <xacro:arg name="orbbec_astra_pro_enabled" default="false"/>
     <xacro:macro name="volta_robot">
         <!-- Footprint -->
@@ -47,19 +52,24 @@
         <!-- Chassis a.k.a base_link -->
         <link name="base_link">
-            <visual>
+            <visual name="visual_base">
                 <origin xyz="0 0 0" rpy="0 0 0" />
-                <geometry>s
-                    <mesh filename="package://volta_description/meshes/volta.STL"/>
+                <geometry>
+                    <mesh filename="package://volta_description/meshes/volta.dae"/>
                 </geometry>
-                <material name="gray"/>
+            </visual>
+            <visual name="visual_logo">
+                <origin xyz="0 0 0" rpy="0 0 0" />
+                <geometry>
+                    <mesh filename="package://volta_description/meshes/volta_logo.dae"/>
+                </geometry>
             </visual>
             <collision>
                 <origin xyz="0 0 0" rpy="0 0 0" />
                 <geometry>
-                    <mesh filename="package://volta_description/meshes/volta.STL"/>
+                    <mesh filename="package://volta_description/meshes/volta.dae"/>
                 </geometry>
             </collision>
             <inertial>
-                <origin xyz ="-0.0223 0.0000 0.1018"/>
+		            <origin xyz ="0.00701 0.0000 0.08382"/>
                 <mass value="${base_mass}"/>
                 <inertia ixx="${base_ixx}" ixy="${base_ixy}" ixz="${base_ixz}" iyy="${base_iyy}" iyz="${base_iyz}" izz="${base_izz}"/>
@@ -73,130 +83,17 @@
             <origin xyz="0.0 ${wheel_joint_y_abs} ${wheel_joint_z_abs}" rpy="0 0 0" />
         </xacro:volta_wheel>
-        <link name="caster_front_left_link">
-            <visual>
-                <origin rpy="0 0 0" xyz="0.0 0.0 0.0"/>
-                <geometry>
-                    <sphere radius="${caster_radius}"/>
-                </geometry>
-                <material name="Black"/>
-            </visual>
-            <collision>
-                <geometry>
-                    <sphere radius="${caster_radius}"/>
-                </geometry>
-                <origin rpy="0 0 0" xyz="0 0 0"/>
-            </collision>
-            <inertial>
-                <mass value="0.5"/>
-                <origin xyz="0 0 0"/>
-                <inertia ixx="0.001" ixy="0.0" ixz="0.0" iyy="0.001" iyz="0.0" izz="0.001"/>
-            </inertial>
-        </link>
-        <joint name="caster_front_left_joint" type="fixed">
-            <parent link="base_link"/>
-            <child link="caster_front_left_link"/>
-            <origin rpy="0 0 0" xyz="${caster_joint_x} ${caster_joint_y} ${caster_joint_z}"/>
-        </joint>
-        <gazebo reference="caster_front_left_link">
-            <turnGravityOff>false</turnGravityOff>
-            <mu1 value="0.0"/>
-            <mu2 value="0.0"/>
-        </gazebo>
-        <link name="caster_front_right_link">
-            <visual>
-                <origin rpy="0 0 0" xyz="0.0 0.0 0.0"/>
-                <geometry>
-                    <sphere radius="${caster_radius}"/>
-                </geometry>
-                <material name="Black"/>
-            </visual>
-            <collision>
-                <geometry>
-                    <sphere radius="${caster_radius}"/>
-                </geometry>
-                <origin rpy="0 0 0" xyz="0 0 0"/>
-            </collision>
-            <inertial>
-                <mass value="0.5"/>
-                <origin xyz="0 0 0"/>
-                <inertia ixx="0.001" ixy="0.0" ixz="0.0" iyy="0.001" iyz="0.0" izz="0.001"/>
-            </inertial>
-        </link>
-        <joint name="caster_front_right_joint" type="fixed">
-            <parent link="base_link"/>
-            <child link="caster_front_right_link"/>
-            <origin rpy="0 0 0" xyz="${caster_joint_x} ${-caster_joint_y} ${caster_joint_z}"/>
-        </joint>
-        <gazebo reference="caster_front_right_link">
-            <turnGravityOff>false</turnGravityOff>
-            <mu1 value="0.0"/>
-            <mu2 value="0.0"/>
-        </gazebo>
-        <link name="caster_rear_right_link">
-            <visual>
-                <origin rpy="0 0 0" xyz="0.0 0.0 0.0"/>
-                <geometry>
-                    <sphere radius="${caster_radius}"/>
-                </geometry>
-                <material name="Black"/>
-            </visual>
-            <collision>
-                <geometry>
-                    <sphere radius="${caster_radius}"/>
-                </geometry>
-                <origin rpy="0 0 0" xyz="0 0 0"/>
-            </collision>
-            <inertial>
-                <mass value="0.5"/>
-                <origin xyz="0 0 0"/>
-                <inertia ixx="0.001" ixy="0.0" ixz="0.0" iyy="0.001" iyz="0.0" izz="0.001"/>
-            </inertial>
-        </link>
-        <joint name="caster_rear_right_joint" type="fixed">
-            <parent link="base_link"/>
-            <child link="caster_rear_right_link"/>
-            <origin rpy="0 0 0" xyz="${-caster_joint_x} ${-caster_joint_y} ${caster_joint_z}"/>
-        </joint>
-        <gazebo reference="caster_rear_right_link">
-            <turnGravityOff>false</turnGravityOff>
-            <mu1 value="0.0"/>
-            <mu2 value="0.0"/>
-        </gazebo>
-        <link name="caster_rear_left_link">
-            <visual>
-                <origin rpy="0 0 0" xyz="0.0 0.0 0.0"/>
-                <geometry>
-                    <sphere radius="${caster_radius}"/>
-                </geometry>
-                <material name="Black"/>
-            </visual>
-            <collision>
-                <geometry>
-                    <sphere radius="${caster_radius}"/>
-                </geometry>
-                <origin rpy="0 0 0" xyz="0 0 0"/>
-            </collision>
-            <inertial>
-                <mass value="0.5"/>
-                <origin xyz="0 0 0"/>
-                <inertia ixx="0.001" ixy="0.0" ixz="0.0" iyy="0.001" iyz="0.0" izz="0.001"/>
-            </inertial>
-        </link>
-        <joint name="caster_rear_left_joint" type="fixed">
-            <parent link="base_link"/>
-            <child link="caster_rear_left_link"/>
-            <origin rpy="0 0 0" xyz="${-caster_joint_x} ${caster_joint_y} ${caster_joint_z}"/>
-        </joint>
-        <gazebo reference="caster_rear_left_link">
-            <turnGravityOff>false</turnGravityOff>
-            <mu1 value="0.0"/>
-            <mu2 value="0.0"/>
-        </gazebo>
-        <gazebo>
-            <plugin name="gazebo_ros_control" filename="libgazebo_ros_control.so">
-                <robotNamespace>$(arg robot_namespace)</robotNamespace>
-                <robotSimType>gazebo_ros_control/DefaultRobotHWSim</robotSimType>
-            </plugin>
-        </gazebo>
+        <!-- Caster wheels -->
+        <xacro:volta_caster caster_prefix="front_left">
+            <origin xyz="${caster_joint_x} ${caster_joint_y} ${caster_joint_z}" rpy="0 0 0" />
+        </xacro:volta_caster>
+        <xacro:volta_caster caster_prefix="front_right">
+            <origin xyz="${caster_joint_x} ${-caster_joint_y} ${caster_joint_z}" rpy="0 0 0" />
+        </xacro:volta_caster>
+        <xacro:volta_caster caster_prefix="rear_right">
+            <origin xyz="${-caster_joint_x} ${-caster_joint_y} ${caster_joint_z}" rpy="0 0 0" />
+        </xacro:volta_caster>
+        <xacro:volta_caster caster_prefix="rear_left">
+            <origin xyz="${-caster_joint_x} ${caster_joint_y} ${caster_joint_z}" rpy="0 0 0" />
+        </xacro:volta_caster>
         <!-- IMU -->
         <xacro:if value="$(arg imu_enabled)">
@@ -206,12 +103,19 @@
         <!-- LIDAR -->
         <xacro:if value="$(arg lidar_enabled)">
-            <xacro:include filename="$(find volta_description)/urdf/accessories/rpi_a3_volta.urdf.xacro"/>
-            <xacro:lidar robot_namespace="$(arg robot_namespace)"></xacro:lidar>
+            <xacro:include filename="$(find volta_description)/urdf/accessories/lidar_volta.urdf.xacro"/>
+            <xacro:lidar rplidar_a3_enabled="$(arg rplidar_a3_enabled)" hokuyo_ust_10lx_enabled="$(arg hokuyo_ust_10lx_enabled)" robot_namespace="$(arg robot_namespace)">  </xacro:lidar>
         </xacro:if>
         <!-- Camera -->
         <xacro:if value="$(arg camera_enabled)">
             <xacro:include filename="$(find volta_description)/urdf/accessories/camera_volta.urdf.xacro"/>
-            <xacro:camera_></xacro:camera_>
+            <xacro:camera_ intel_d435i_enabled="$(arg intel_d435i_enabled)" orbbec_astra_pro_enabled="$(arg orbbec_astra_pro_enabled)" robot_namespace="$(arg robot_namespace)"></xacro:camera_>
         </xacro:if>
+        <!-- Robot Gazebo tag -->
+        <gazebo>
+            <plugin name="gazebo_ros_control" filename="libgazebo_ros_control.so">
+                <robotNamespace>$(arg robot_namespace)</robotNamespace>
+                <robotSimType>gazebo_ros_control/DefaultRobotHWSim</robotSimType>
+            </plugin>
+        </gazebo>
     </xacro:macro>
 </robot>

File: volta_description/urdf/volta_properties.xacro (robot description, xacro)
@@ -28,42 +28,54 @@
         <color rgba="0 0 0.8 1"/>
     </material>
-    <material name="white">
-       <color rgba="1 1 1 1"/>
+    <material name="silver">
+       <color rgba="0.75 0.75 0.75 1"/>
     </material>
-    <material name="gray">
-        <color rgba="0.5 0.5 0.5 1"/>
+    <material name="grey">
+       <color rgba="0.824 0.824 0.824 1"/>
     </material>
-    <xacro:property name="base_underside_h" value="0.03275"/>
-    <xacro:property name="base_mass" value="15.0000"/>
-    <xacro:property name="base_l" value="0.4000"/>
-    <xacro:property name="base_w" value="0.3200"/>
-    <xacro:property name="base_h" value="0.2295"/>
-    <xacro:property name="base_ixx" value="0.1815"/>
-    <xacro:property name="base_ixy" value="0.0000"/>
-    <xacro:property name="base_ixz" value="-0.0158"/>
-    <xacro:property name="base_iyy" value="0.2238"/>
-    <xacro:property name="base_iyz" value="0.0000"/>
-    <xacro:property name="base_izz" value="0.2856"/>
-    <xacro:property name="wheel_mass" value="0.0563"/>
+    <material name="black">
+	     <color rgba="0.260 0.260 0.300 1"/>
+    </material>
+    <material name="orange">
+	     <color rgba="0.999 0.547 0 1"/>
+    </material>
+    <material name="red">
+	     <color rgba="0.543 0 0 1"/>
+    </material>
+    <xacro:property name="base_underside_h" value="0.035"/>
+    <xacro:property name="base_mass" value="20.0000"/>
+    <xacro:property name="base_l" value="0.4950"/>
+    <xacro:property name="base_w" value="0.3650"/>
+    <xacro:property name="base_h" value="0.21905"/>
+    <!-- Volta R2 -->
+    <xacro:property name="base_ixx" value="0.41802"/>
+    <xacro:property name="base_ixy" value="0"/>
+    <xacro:property name="base_ixz" value="0.00305"/>
+    <xacro:property name="base_iyy" value="0.50105"/>
+    <xacro:property name="base_iyz" value="0"/>
+    <xacro:property name="base_izz" value="0.60276"/>
+    <!-- Volta_R1 -->
+    <xacro:property name="wheel_mass" value="0.5"/>
     <xacro:property name="wheel_width" value="0.020" />
-    <xacro:property name="wheel_radius" value="0.035" />
-    <xacro:property name="wheel_joint_y_abs" value="0.1425" />
-    <xacro:property name="wheel_joint_z_abs" value="0.0215" />
-    <xacro:property name="wheel_ixx" value="0.001"/>
+    <xacro:property name="wheel_radius" value="0.0425" />
+    <xacro:property name="wheel_joint_y_abs" value="0.1604" />
+    <xacro:property name="wheel_joint_z_abs" value="0.02640" />
+    <xacro:property name="wheel_ixx" value="0.0003"/>
     <xacro:property name="wheel_ixy" value="0.000"/>
     <xacro:property name="wheel_ixz" value="0.000"/>
-    <xacro:property name="wheel_iyy" value="0.001"/>
+    <xacro:property name="wheel_iyy" value="0.0005"/>
     <xacro:property name="wheel_iyz" value="0.000"/>
-    <xacro:property name="wheel_izz" value="0.001"/>
-    <xacro:property name="caster_radius" value="0.016"/>
-    <xacro:property name="caster_joint_x" value="0.1200"/>
-    <xacro:property name="caster_joint_y" value="0.0950"/>
-    <xacro:property name="caster_joint_z" value="0.006"/>
-    <xacro:property name="lidar_joint_x" value="0.1200"/>
+    <xacro:property name="wheel_izz" value="0.0003"/>
+    <xacro:property name="caster_radius" value="0.015"/>
+    <xacro:property name="caster_joint_x" value="0.15925"/>
+    <xacro:property name="caster_joint_y" value="0.1210"/>
+    <xacro:property name="caster_joint_z" value="-0.0008"/>
+    <!-- base of lidar mopunt, x position in lidar_volta.urdf.xacro -->
     <xacro:property name="lidar_joint_y" value="0.0"/>
-    <xacro:property name="lidar_joint_z" value="0.15"/>
-    <xacro:property name="camera_joint_x" value="0.1595"/>
+    <xacro:property name="lidar_joint_z" value="0.1140"/>
+    <!-- base of camera mount -->
+    <xacro:property name="camera_joint_x" value="0.2285"/>
     <xacro:property name="camera_joint_y" value="0.0000"/>
-    <xacro:property name="camera_joint_z" value="0.1840"/>
+    <xacro:property name="camera_joint_z" value="0.1935"/>
     <xacro:property name="dummy_inertia" value="1e-09"/>
 </robot>
