Commit message: Noetic-devel initial commit.

File: volta_description/urdf/accessories/camera_volta.urdf.xacro (robot description, xacro)
@@ -1,5 +1,5 @@
 <?xml version="1.0"?>
 <!--
-Copyright (c) 2020, Botsync Pte. Ltd.
+Copyright (c) 2021, Botsync Pte. Ltd.
 All rights reserved.
 Redistribution and use in source and binary forms, with or without

File: volta_description/urdf/accessories/imu_volta.urdf.xacro (robot description, xacro)
@@ -1,5 +1,5 @@
 <?xml version="1.0"?>
 <!--
-Copyright (c) 2020, Botsync Pte. Ltd.
+Copyright (c) 2021, Botsync Pte. Ltd.
 All rights reserved.
 Redistribution and use in source and binary forms, with or without

File: volta_description/urdf/accessories/lidar_volta.urdf.xacro (robot description, xacro)
@@ -1,5 +1,5 @@
 <?xml version="1.0"?>
 <!--
-Copyright (c) 2020, Botsync Pte. Ltd.
+Copyright (c) 2021, Botsync Pte. Ltd.
 All rights reserved.
 Redistribution and use in source and binary forms, with or without

File: volta_description/urdf/components/caster_volta.urdf.xacro (robot description, xacro)
@@ -1,5 +1,5 @@
 <?xml version="1.0"?>
 <!--
-Copyright (c) 2020, Botsync Pte. Ltd.
+Copyright (c) 2021, Botsync Pte. Ltd.
 All rights reserved.
 Redistribution and use in source and binary forms, with or without
@@ -34,5 +34,5 @@
                     <sphere radius="${caster_radius}"/>
                 </geometry>
-                <material name="Black"/>
+                <material name="black"/>
             </visual>
             <collision>

File: volta_description/urdf/components/wheel_volta.urdf.xacro (robot description, xacro)
@@ -1,5 +1,5 @@
 <?xml version="1.0"?>
 <!--
-Copyright (c) 2020, Botsync Pte. Ltd.
+Copyright (c) 2021, Botsync Pte. Ltd.
 All rights reserved.
 Redistribution and use in source and binary forms, with or without

File: volta_description/urdf/volta.urdf.xacro (robot description, xacro)
@@ -1,5 +1,5 @@
 <?xml version="1.0"?>
 <!--
-Copyright (c) 2020, Botsync Pte. Ltd.
+Copyright (c) 2021, Botsync Pte. Ltd.
 All rights reserved.
 Redistribution and use in source and binary forms, with or without

File: volta_description/urdf/volta.xacro (robot description, xacro)
@@ -1,4 +1,4 @@
 <!--
-Copyright (c) 2020, Botsync Pte. Ltd.
+Copyright (c) 2021, Botsync Pte. Ltd.
 All rights reserved.
 Redistribution and use in source and binary forms, with or without

File: volta_description/urdf/volta_properties.xacro (robot description, xacro)
@@ -1,5 +1,5 @@
 <?xml version="1.0"?>
 <!--
-Copyright (c) 2020, Botsync Pte. Ltd.
+Copyright (c) 2021, Botsync Pte. Ltd.
 All rights reserved.
 Redistribution and use in source and binary forms, with or without
